Commit message: minimum working example with robot commander and panda

File: ace_ws/src/panda_resources/panda_description/urdf/panda.urdf (robot description, URDF)
Before this commit: robot panda, 12 links, 11 joints
Links:
- link panda_hand: geometry collision mesh filename=package://panda_description/meshes/collision/hand.stl; visual mesh filename=package://panda_description/meshes/visual/hand.dae
- link panda_leftfinger: geometry collision mesh filename=package://panda_description/meshes/collision/finger.stl; visual mesh filename=package://panda_description/meshes/visual/finger.dae
- link panda_link0: geometry collision mesh filename=package://panda_description/meshes/collision/link0.stl; visual mesh filename=package://panda_description/meshes/visual/link0.dae
- link panda_link1: geometry collision mesh filename=package://panda_description/meshes/collision/link1.stl; visual mesh filename=package://panda_description/meshes/visual/link1.dae
- link panda_link2: geometry collision mesh filename=package://panda_description/meshes/collision/link2.stl; visual mesh filename=package://panda_description/meshes/visual/link2.dae
- link panda_link3: geometry collision mesh filename=package://panda_description/meshes/collision/link3.stl; visual mesh filename=package://panda_description/meshes/visual/link3.dae
- link panda_link4: geometry collision mesh filename=package://panda_description/meshes/collision/link4.stl; visual mesh filename=package://panda_description/meshes/visual/link4.dae
- link panda_link5: geometry collision mesh filename=package://panda_description/meshes/collision/link5.stl; visual mesh filename=package://panda_description/meshes/visual/link5.dae
- link panda_link6: geometry collision mesh filename=package://panda_description/meshes/collision/link6.stl; visual mesh filename=package://panda_description/meshes/visual/link6.dae
- link panda_link7: geometry collision mesh filename=package://panda_description/meshes/collision/link7.stl; visual mesh filename=package://panda_description/meshes/visual/link7.dae
- link panda_rightfinger: geometry collision mesh filename=package://panda_description/meshes/collision/finger.stl; visual mesh filename=package://panda_description/meshes/visual/finger.dae

File: ace_ws/src/panda_resources/panda_description/urdf/panda.urdf.xacro (robot description, xacro)
@@ -8,10 +8,10 @@
         <visual>
             <geometry>
-                <mesh filename="file://$(find moveit_resources_panda_description)/meshes/visual/link0.dae" />
-            </geometry>
-        </visual>
-        <collision>
-            <geometry>
-                <mesh filename="file://$(find moveit_resources_panda_description)/meshes/collision/link0.stl" />
+                <mesh filename="file://$(find panda_description)/meshes/visual/link0.dae" />
+            </geometry>
+        </visual>
+        <collision>
+            <geometry>
+                <mesh filename="file://$(find panda_description)/meshes/collision/link0.stl" />
             </geometry>
         </collision>
@@ -25,10 +25,10 @@
         <visual>
             <geometry>
-                <mesh filename="file://$(find moveit_resources_panda_description)/meshes/visual/link1.dae" />
-            </geometry>
-        </visual>
-        <collision>
-            <geometry>
-                <mesh filename="file://$(find moveit_resources_panda_description)/meshes/collision/link1.stl" />
+                <mesh filename="file://$(find panda_description)/meshes/visual/link1.dae" />
+            </geometry>
+        </visual>
+        <collision>
+            <geometry>
+                <mesh filename="file://$(find panda_description)/meshes/collision/link1.stl" />
             </geometry>
         </collision>
@@ -51,10 +51,10 @@
         <visual>
             <geometry>
-                <mesh filename="file://$(find moveit_resources_panda_description)/meshes/visual/link2.dae" />
-            </geometry>
-        </visual>
-        <collision>
-            <geometry>
-                <mesh filename="file://$(find moveit_resources_panda_description)/meshes/collision/link2.stl" />
+                <mesh filename="file://$(find panda_description)/meshes/visual/link2.dae" />
+            </geometry>
+        </visual>
+        <collision>
+            <geometry>
+                <mesh filename="file://$(find panda_description)/meshes/collision/link2.stl" />
             </geometry>
         </collision>
@@ -77,10 +77,10 @@
         <visual>
             <geometry>
-                <mesh filename="file://$(find moveit_resources_panda_description)/meshes/visual/link3.dae" />
-            </geometry>
-        </visual>
-        <collision>
-            <geometry>
-                <mesh filename="file://$(find moveit_resources_panda_description)/meshes/collision/link3.stl" />
+                <mesh filename="file://$(find panda_description)/meshes/visual/link3.dae" />
+            </geometry>
+        </visual>
+        <collision>
+            <geometry>
+                <mesh filename="file://$(find panda_description)/meshes/collision/link3.stl" />
             </geometry>
         </collision>
@@ -103,10 +103,10 @@
         <visual>
             <geometry>
-                <mesh filename="file://$(find moveit_resources_panda_description)/meshes/visual/link4.dae" />
-            </geometry>
-        </visual>
-        <collision>
-            <geometry>
-                <mesh filename="file://$(find moveit_resources_panda_description)/meshes/collision/link4.stl" />
+                <mesh filename="file://$(find panda_description)/meshes/visual/link4.dae" />
+            </geometry>
+        </visual>
+        <collision>
+            <geometry>
+                <mesh filename="file://$(find panda_description)/meshes/collision/link4.stl" />
             </geometry>
         </collision>
@@ -129,10 +129,10 @@
         <visual>
             <geometry>
-                <mesh filename="file://$(find moveit_resources_panda_description)/meshes/visual/link5.dae" />
-            </geometry>
-        </visual>
-        <collision>
-            <geometry>
-                <mesh filename="file://$(find moveit_resources_panda_description)/meshes/collision/link5.stl" />
+                <mesh filename="file://$(find panda_description)/meshes/visual/link5.dae" />
+            </geometry>
+        </visual>
+        <collision>
+            <geometry>
+                <mesh filename="file://$(find panda_description)/meshes/collision/link5.stl" />
             </geometry>
         </collision>
@@ -155,10 +155,10 @@
         <visual>
             <geometry>
-                <mesh filename="file://$(find moveit_resources_panda_description)/meshes/visual/link6.dae" />
-            </geometry>
-        </visual>
-        <collision>
-            <geometry>
-                <mesh filename="file://$(find moveit_resources_panda_description)/meshes/collision/link6.stl" />
+                <mesh filename="file://$(find panda_description)/meshes/visual/link6.dae" />
+            </geometry>
+        </visual>
+        <collision>
+            <geometry>
+                <mesh filename="file://$(find panda_description)/meshes/collision/link6.stl" />
             </geometry>
         </collision>
@@ -181,10 +181,10 @@
         <visual>
             <geometry>
-                <mesh filename="file://$(find moveit_resources_panda_description)/meshes/visual/link7.dae" />
-            </geometry>
-        </visual>
-        <collision>
-            <geometry>
-                <mesh filename="file://$(find moveit_resources_panda_description)/meshes/collision/link7.stl" />
+                <mesh filename="file://$(find panda_description)/meshes/visual/link7.dae" />
+            </geometry>
+        </visual>
+        <collision>
+            <geometry>
+                <mesh filename="file://$(find panda_description)/meshes/collision/link7.stl" />
             </geometry>
         </collision>
@@ -219,10 +219,10 @@
         <visual>
             <geometry>
-                <mesh filename="file://$(find moveit_resources_panda_description)/meshes/visual/hand.dae" />
-            </geometry>
-        </visual>
-        <collision>
-            <geometry>
-                <mesh filename="file://$(find moveit_resources_panda_description)/meshes/collision/hand.stl" />
+                <mesh filename="file://$(find panda_description)/meshes/visual/hand.dae" />
+            </geometry>
+        </visual>
+        <collision>
+            <geometry>
+                <mesh filename="file://$(find panda_description)/meshes/collision/hand.stl" />
             </geometry>
         </collision>
@@ -236,10 +236,10 @@
         <visual>
             <geometry>
-                <mesh filename="file://$(find moveit_resources_panda_description)/meshes/visual/finger.dae" />
-            </geometry>
-        </visual>
-        <collision>
-            <geometry>
-                <mesh filename="file://$(find moveit_resources_panda_description)/meshes/collision/finger.stl" />
+                <mesh filename="file://$(find panda_description)/meshes/visual/finger.dae" />
+            </geometry>
+        </visual>
+        <collision>
+            <geometry>
+                <mesh filename="file://$(find panda_description)/meshes/collision/finger.stl" />
             </geometry>
         </collision>
@@ -254,5 +254,5 @@
             <origin rpy="0 0 3.14159265359" xyz="0 0 0" />
             <geometry>
-                <mesh filename="file://$(find moveit_resources_panda_description)/meshes/visual/finger.dae" />
+                <mesh filename="file://$(find panda_description)/meshes/visual/finger.dae" />
             </geometry>
         </visual>
@@ -260,5 +260,5 @@
             <origin rpy="0 0 3.14159265359" xyz="0 0 0" />
             <geometry>
-                <mesh filename="file://$(find moveit_resources_panda_description)/meshes/collision/finger.stl" />
+                <mesh filename="file://$(find panda_description)/meshes/collision/finger.stl" />
             </geometry>
         </collision>

File: ace_ws/src/panda_resources/panda_moveit_config/config/panda.urdf.xacro (robot description, xacro)
@@ -4,5 +4,5 @@
     <xacro:arg name="ros2_control_hardware_type" default="mock_components" />
     <!-- Import panda urdf file -->
-    <xacro:include filename="$(find moveit_resources_panda_description)/urdf/panda.urdf.xacro" />
+    <xacro:include filename="$(find panda_description)/urdf/panda.urdf.xacro" />
     <!-- Import panda ros2_control description -->
     <xacro:include filename="panda.ros2_control.xacro" />

File: ace_ws/src/panda_resources/panda_moveit_config/config/panda_arm.srdf.xacro (robot description, xacro)
@@ -5,5 +5,5 @@
 -->
 <robot xmlns:xacro="http://www.ros.org/wiki/xacro" name="panda">
-  <xacro:include filename="$(find moveit_resources_panda_moveit_config)/config/panda_arm.xacro" />
+  <xacro:include filename="$(find panda_moveit_config)/config/panda_arm.xacro" />
   <xacro:panda_arm />
 </robot>

File: ace_ws/src/panda_resources/panda_moveit_config/config/panda_arm_hand.srdf.xacro (robot description, xacro)
@@ -5,6 +5,6 @@
 -->
 <robot xmlns:xacro="http://www.ros.org/wiki/xacro" name="panda">
-  <xacro:include filename="$(find moveit_resources_panda_moveit_config)/config/panda_arm.xacro" />
-  <xacro:include filename="$(find moveit_resources_panda_moveit_config)/config/hand.xacro" />
+  <xacro:include filename="$(find panda_moveit_config)/config/panda_arm.xacro" />
+  <xacro:include filename="$(find panda_moveit_config)/config/hand.xacro" />
   <xacro:panda_arm />
   <xacro:hand />
