Commit message: fixed gz_frame_id for camera, it works now!

File: ace_ws/src/ur_simulation_gz/urdf/rgbd.xacro (robot description, xacro)
@@ -1,10 +1,19 @@
 <?xml version="1.0"?>
 <robot xmlns:xacro="http://www.ros.org/wiki/xacro" >
+    <xacro:macro name="inertial_cylinder" params="mass length radius *origin">
+        <inertial>
+            <xacro:insert_block name="origin"/>
+            <mass value="${mass}" />
+            <inertia ixx="${(1/12) * mass * (3*radius*radius + length*length)}" ixy="0.0" ixz="0.0"
+                    iyy="${(1/12) * mass * (3*radius*radius + length*length)}" iyz="0.0"
+                    izz="${(1/2) * mass * (radius*radius)}" />
+        </inertial>
+    </xacro:macro>
     <joint name="cam_joint" type="fixed">
         <parent link="wrist_3_link"/>
-        <child link="cam_frame"/>
+        <child link="rgbd_camera"/>
         <origin xyz="0.1 0 0.175" rpy="0 0 0"/>
     </joint>
-    <link name="cam_frame">
+    <link name="rgbd_camera">
         <visual>
             <geometry>
@@ -22,5 +31,5 @@
         </xacro:inertial_cylinder>
     </link>
-    <gazebo reference="cam_frame">
+    <gazebo reference="rgbd_camera">
         <material>Gazebo/Red</material>
         <sensor name="rgbd_camera" type="rgbd_camera">
@@ -40,4 +49,6 @@
           <visualize>true</visualize>
           <topic>rgbd_camera</topic>
+        <gz_frame_id>rgbd_camera</gz_frame_id>
+        </sensor>
     </gazebo>
 </robot>

File: ace_ws/src/ur_simulation_gz/urdf/ur_gz.urdf.xacro (robot description, xacro)
@@ -22,5 +22,5 @@
   <xacro:include filename="$(find ur_description)/urdf/ur_macro.xacro"/>
   <xacro:include filename="$(find ur_simulation_gz)/urdf/ur_gz.ros2_control.xacro" />
-  <!--xacro:include filename="$(find ur_simulation_gz)/urdf/rgbd.xacro" /-->
+  <xacro:include filename="$(find ur_simulation_gz)/urdf/rgbd.xacro" />
   <!-- possible 'ur_type' values: ur3, ur3e, ur5, ur5e, ur10, ur10e, ur16e, ur20, ur30 -->
   <!-- the default value should raise an error in case this was called without defining the type -->

Commit message: added kimect mesh, cmaere currently filming in x direction

File: ace_ws/src/ur_simulation_gz/urdf/rgbd.xacro (robot description, xacro)
@@ -13,24 +13,26 @@
         <parent link="wrist_3_link"/>
         <child link="rgbd_camera"/>
-        <origin xyz="0.1 0 0.175" rpy="0 0 0"/>
+        <origin xyz="0.0 -0.02 0.0" rpy="0 -1.5707 1.5707"/>
     </joint>
     <link name="rgbd_camera">
         <visual>
-            <geometry>
-                <cylinder radius="0.05" length="0.04"/>
-            </geometry>
-            <material name="red"/>
+        <origin xyz="0 0 0" rpy="0 0 1.5707"/>
+        <geometry>
+            <mesh filename="file:///home/lisa/master_thesis/ace_ws/src/ur_simulation_gz/kinect.dae"/>
+        </geometry>
         </visual>
         <collision>
+            <origin xyz="0.0 0.0 0.0" rpy="0 0 0"/>
             <geometry>
-                <cylinder radius="0.05" length="0.04"/>
+                <box size="0.07271 0.27794 0.073"/>
             </geometry>
         </collision>
-        <xacro:inertial_cylinder mass="0.1" length="0.04" radius="0.05">
-            <origin xyz="0 0 0" rpy="0 0 0"/>
-        </xacro:inertial_cylinder>
+        <inertial>
+            <mass value="0.001" />
+            <origin xyz="0 0 0" />
+            <inertia ixx="0.0001" ixy="0.0" ixz="0.0" iyy="0.0001" iyz="0.0" izz="0.0001" />
+        </inertial>
     </link>
     <gazebo reference="rgbd_camera">
-        <material>Gazebo/Red</material>
         <sensor name="rgbd_camera" type="rgbd_camera">
           <camera>
