Commit message: added camera but still a few  bugs

File: ace_ws/src/ur_moveit_config/srdf/ur_macro.srdf.xacro (robot description, xacro)
@@ -54,3 +54,4 @@
     <disable_collisions link1="wrist_2_link" link2="wrist_3_link" reason="Adjacent" />
   </xacro:macro>
+   <!--Kinect-->
 </robot>

File: ace_ws/src/ur_simulation_gz/urdf/ur_gz.urdf.xacro (robot description, xacro)
@@ -51,3 +51,163 @@
     transmission_hw_interface="$(arg transmission_hw_interface)"
   />
+  <!--gazebo>
+      <plugin
+      filename="gz-sim-physics-system"
+      name="gz::sim::systems::Physics">
+    </plugin>
+  </gazebo-->
+ <gazebo>
+    <plugin filename="gz-sim-sensors-system" name="gz::sim::systems::Sensors">
+    </plugin>
+  </gazebo>
+   <gazebo>
+    <plugin filename="gz-sim-scene-broadcaster-system" name="gz::sim::systems::SceneBroadcaster">
+    </plugin>
+  </gazebo>
+   <joint name="laser_joint" type="fixed">
+        <parent link="wrist_3_link"/>
+        <child link="laser_frame"/>
+        <origin xyz="0.1 0 0.175" rpy="0 0 0"/>
+    </joint>
+    <link name="laser_frame">
+        <inertial>
+          <mass>0.1</mass>
+          <inertia>
+            <ixx>0.000166667</ixx>
+            <iyy>0.000166667</iyy>
+            <izz>0.000166667</izz>
+          </inertia>
+        </inertial>
+        <collision name="collision">
+          <geometry>
+            <box>
+              <size>0.1 0.1 0.1</size>
+            </box>
+          </geometry>
+        </collision>
+        <visual name="visual">
+          <geometry>
+            <box>
+              <size>2 2 2</size>
+            </box>
+          </geometry>
+        </visual>
+    </link>
+    <gazebo reference="laser_frame">
+        <sensor name="rgbd_camera" type="rgbd_camera">
+          <camera>
+            <horizontal_fov>1.047</horizontal_fov>
+            <image>
+              <width>320</width>
+              <height>240</height>
+            </image>
+            <clip>
+              <near>0.1</near>
+              <far>100</far>
+            </clip>
+          </camera>
+          <always_on>1</always_on>
+          <update_rate>30</update_rate>
+          <visualize>true</visualize>
+          <topic>rgbd_camera</topic>
+          <enable_metrics>true</enable_metrics>
+        </sensor>
+    </gazebo>
+      <!--link name="cam_mount">
+        <pose>0.05 0.05 0.05 0 0 0</pose>
+        <inertial>
+          <mass value="0.1"/>
+          <inertia ixx="0.1" ixy="0" ixz="0" iyy="0.1" iyz="0" izz="0.1"/>
+        </inertial>
+        <visual>
+        <origin xyz="0 0 0" rpy="0 0 0" />
+        <geometry>
+          <box size="1 1 1" />
+        </geometry>
+        <material name="Cyan">
+          <color rgba="0 1.0 1.0 1.0"/>
+        </material>
+        </visual>
+        <collision>
+          <origin xyz="0 0 0" rpy="0 0 0"/>
+          <geometry>
+            <cylinder radius="1" length="0.5"/>
+          </geometry>
+        </collision>
+        <sensor name="rgbd_camera" type="rgbd_camera">
+          <camera>
+            <horizontal_fov>1.047</horizontal_fov>
+            <image>
+              <width>320</width>
+              <height>240</height>
+            </image>
+            <clip>
+              <near>0.1</near>
+              <far>100</far>
+            </clip>
+          </camera>
+          <always_on>1</always_on>
+          <update_rate>30</update_rate>
+          <visualize>true</visualize>
+          <topic>rgbd_camera</topic>
+          <enable_metrics>true</enable_metrics>
+        </sensor>
+      </link-->
+      <!--joint name="cam_mount_joint" type="fixed">
+          <origin xyz="0 0 1" rpy="0 0 0"/>
+          <parent link="wrist_3_link"/>
+          <child link="cam_mount"/>
+       </joint-->
+   <!--model name="custom_params">
+      <pose>5 0 0.5 0 0.0 3.14</pose>
+      <link name="link">
+        <pose>0.05 0.05 0.05 0 0 0</pose>
+        <inertial>
+          <mass>0.1</mass>
+          <inertia>
+            <ixx>0.000166667</ixx>
+            <iyy>0.000166667</iyy>
+            <izz>0.000166667</izz>
+          </inertia>
+        </inertial>
+        <collision name="collision">
+          <geometry>
+            <box>
+              <size>0.1 0.1 0.1</size>
+            </box>
+          </geometry>
+        </collision>
+        <visual name="visual">
+          <geometry>
+            <box>
+              <size>0.1 0.1 0.1</size>
+            </box>
+          </geometry>
+        </visual>
+        <sensor name="depth_camera" type="depth_camera">
+          <camera>
+            <horizontal_fov>1.047</horizontal_fov>
+            <image>
+              <width>320</width>
+              <height>240</height>
+              <format>R_FLOAT32</format>
+            </image>
+            <clip>
+              <near>0.1</near>
+              <far>100</far>
+            </clip>
+          </camera>
+          <always_on>1</always_on>
+          <update_rate>10</update_rate>
+          <visualize>true</visualize>
+          <topic>depth_camera</topic>
+          <plugin
+            filename="RosGzPointCloud"
+            name="ros_gz_point_cloud::PointCloud">
+            <topic>points</topic>
+            <frame_id>map</frame_id>
+          </plugin>
+        </sensor>
+      </link>
+    </model-->
 </robot>

Commit message: Filtered collision between camera and wrist3

File: ace_ws/src/ur_moveit_config/srdf/ur_macro.srdf.xacro (robot description, xacro)
@@ -53,4 +53,5 @@
     <disable_collisions link1="wrist_1_link" link2="wrist_3_link" reason="Never" />
     <disable_collisions link1="wrist_2_link" link2="wrist_3_link" reason="Adjacent" />
+    <disable_collisions link1="wrist_3_link" link2="rgbd_camera" reason="Adjacent" />
   </xacro:macro>
    <!--Kinect-->

File: ace_ws/src/ur_simulation_gz/urdf/rgbd.xacro (robot description, xacro)
@@ -13,5 +13,5 @@
         <parent link="wrist_3_link"/>
         <child link="rgbd_camera"/>
-        <origin xyz="0.0 -0.02 0.0" rpy="0 -1.5707 1.5707"/>
+        <origin xyz="0.0 -0.05 0.0" rpy="0 -1.5707 1.5707"/>
     </joint>
     <link name="rgbd_camera">

Commit message: linked robot to table, adding complex objects slows down rtf

File: ace_ws/src/ur_moveit_config/srdf/ur_macro.srdf.xacro (robot description, xacro)
@@ -55,4 +55,5 @@
     <disable_collisions link1="wrist_2_link" link2="wrist_3_link" reason="Adjacent" />
     <disable_collisions link1="wrist_3_link" link2="rgbd_camera" reason="Adjacent" />
+    <disable_collisions link1="base_link" link2="table_link" reason="Adjacent" />
   </xacro:macro>
    <!--Kinect-->

File: ace_ws/src/ur_simulation_gz/urdf/rgbd.xacro (robot description, xacro)
@@ -19,5 +19,5 @@
         <origin xyz="0 0 0" rpy="0 0 1.5707"/>
         <geometry>
-            <mesh filename="file:///home/lisa/master_thesis/ace_ws/src/ur_simulation_gz/kinect.dae"/>
+            <mesh filename="file:///home/lisa/master_thesis/ace_ws/src/ur_simulation_gz/material/kinect.dae"/>
         </geometry>
         </visual>

File: ace_ws/src/ur_simulation_gz/urdf/ur_gz.urdf.xacro (robot description, xacro)
@@ -39,9 +39,16 @@
   <!-- create link fixed to the "world" -->
   <link name="world" />
+  <link name="table_link" />
+    <!-- Add a fixed joint to attach the table to the world -->
+  <joint name="world_to_table" type="fixed">
+    <parent link="world"/>
+    <child link="table_link"/>
+    <origin xyz="0 0 .755" rpy="0 0 0"/>
+  </joint>
   <!-- arm -->
   <xacro:ur_robot
     name="$(arg name)"
     tf_prefix="$(arg tf_prefix)"
-    parent="world"
+    parent="table_link"
     joint_limits_parameters_file="$(arg joint_limit_params)"
     kinematics_parameters_file="$(arg kinematics_params)"
